File: boards/commbrd/commbrd.sch (KiCad schematic (older format))
At the start: 20 parts, among them J1 USB_2, J2 RJ45, J3 RJ45, U1 FT232RL, U2 SN75176B

Commit message: added footprints, part numbers, digikey part numbers
Parts:
- C1, C3: footprint (none) -> SM0805; DigikeyPart (none) -> 311-1361-1-ND; Part (none) -> CC0805ZRY5V9BB104
- C2: footprint (none) -> SM0805; DigikeyPart (none) -> 478-4086-1-ND; Part (none) -> TPSA106M010R1800
- D1: footprint (none) -> SM1206; DigikeyPart (none) -> 754-1142-1-ND; Part (none) -> APT3216SRCPRV
- D2, D3: footprint (none) -> LED-1206; DigikeyPart (none) -> 754-1141-1-ND; Part (none) -> APT3216SGC
- J1: footprint VCC -> USB_MINI_A; Data- D- -> (none); DigikeyPart (none) -> ED90342CT-ND; Ground GND -> (none); Part (none) -> 896-43-005-00-100001
- J2: footprint (none) -> RJ45_8
- J3: footprint (none) -> RJ45_8; DigikeyPart (none) -> WM5572-ND; Part (none) -> 95501-2882
- JP1: footprint (none) -> SM1206; DigikeyPart (none) -> N/A; Part (none) -> N/A
- PGND1, PRXD1, PTXD1, PVCC1: footprint (none) -> SIL-1; DigikeyPart (none) -> N/A; Part (none) -> N/A
- R1, R2, R3: footprint (none) -> SM0805; DigikeyPart (none) -> RMCF0805JT1K00CT-ND; Part (none) -> RMCF0805JT1K00
- R4: footprint (none) -> SM0805; DigikeyPart (none) -> RMCF0805JT120RCT-ND; Part (none) -> RMCF0805JT120R
- U1: footprint (none) -> SSOP28; DigikeyPart (none) -> 768-1007-1-ND; Part (none) -> FT232RL-REEL
- U2: footprint DIL8 -> SOIC8; DigikeyPart (none) -> 296-27995-1-ND; Part (none) -> SN75176BPSR
Changed lines of the file:
@@
-EESchema Schematic File Version 2  date Mon 30 May 2011 04:01:16 AM EDT
+EESchema Schematic File Version 2  date Mon 13 Jun 2011 01:48:36 AM EDT
 LIBS:power
 LIBS:device
@@
 Sheet 1 1
 Title ""
-Date "30 may 2011"
+Date "13 jun 2011"
 Rev ""
 Comp ""
@@
 F 0 "PTXD1" V 6650 2050 40  0000 L CNN
 F 1 "CONN_1" H 6600 2155 30  0001 C CNN
+F 2 "SIL-1" H 6600 2100 60  0001 C CNN
+F 4 "N/A" H 6600 2100 60  0001 C CNN "Part"
+F 5 "N/A" H 6600 2100 60  0001 C CNN "DigikeyPart"
 	1    6600 2100
 	0    -1   -1   0
@@
 F 0 "PRXD1" V 6550 3000 40  0000 L CNN
 F 1 "CONN_1" H 6500 3055 30  0001 C CNN
+F 2 "SIL-1" V 6590 2960 60  0001 C CNN
+F 4 "N/A" H 6500 3000 60  0001 C CNN "Part"
+F 5 "N/A" H 6500 3000 60  0001 C CNN "DigikeyPart"
 	1    6500 3000
 	0    1    1    0
@@
 F 0 "D1" H 2850 3700 50  0000 C CNN
 F 1 "LED" H 2850 3800 50  0000 C CNN
+F 2 "SM1206" H 2800 3750 60  0001 C CNN
+F 4 "APT3216SRCPRV" H 2850 3600 60  0001 C CNN "Part"
+F 5 "754-1142-1-ND" H 2850 3600 60  0001 C CNN "DigikeyPart"
 	1    2850 3600
 	0    1    1    0
@@
 F 0 "R1" V 2930 3100 50  0000 C CNN
 F 1 "1K" V 2850 3100 50  0000 C CNN
+F 2 "SM0805" V 2980 3050 60  0001 C CNN
+F 4 "RMCF0805JT1K00" H 2850 3100 60  0001 C CNN "Part"
+F 5 "RMCF0805JT1K00CT-ND" H 2850 3100 60  0001 C CNN "DigikeyPart"
 	1    2850 3100
 	-1   0    0    1
@@
 F 0 "PGND1" V 3500 3150 40  0000 L CNN
 F 1 "CONN_1" H 3450 3205 30  0001 C CNN
+F 2 "SIL-1" V 3540 3110 60  0001 C CNN
+F 4 "N/A" H 3450 3150 60  0001 C CNN "Part"
+F 5 "N/A" H 3450 3150 60  0001 C CNN "DigikeyPart"
 	1    3450 3150
 	0    1    1    0
@@
 F 0 "PVCC1" V 3500 2150 40  0000 L CNN
 F 1 "CONN_1" H 3450 2205 30  0001 C CNN
+F 2 "SIL-1" V 3540 2110 60  0001 C CNN
+F 4 "N/A" H 3450 2150 60  0001 C CNN "Part"
+F 5 "N/A" H 3450 2150 60  0001 C CNN "DigikeyPart"
 	1    3450 2150
 	0    -1   -1   0
@@
 F 0 "J2" H 9250 3750 60  0000 C CNN
 F 1 "RJ45" H 8900 3750 60  0000 C CNN
+F 2 "RJ45_8" H 9310 3810 60  0001 C CNN
 	1    9050 3250
 	0    1    1    0
@@
 F 0 "J3" H 9250 2750 60  0000 C CNN
 F 1 "RJ45" H 8900 2750 60  0000 C CNN
+F 2 "RJ45_8" H 9310 2810 60  0001 C CNN
+F 4 "95501-2882" H 9050 2250 60  0001 C CNN "Part"
+F 5 "WM5572-ND" H 9050 2250 60  0001 C CNN "DigikeyPart"
 	1    9050 2250
 	0    1    1    0
@@
 F 0 "R4" V 8080 2550 50  0000 C CNN
 F 1 "120" V 8000 2550 50  0000 C CNN
+F 2 "SM0805" V 8130 2500 60  0001 C CNN
+F 4 "RMCF0805JT120R" H 8000 2550 60  0001 C CNN "Part"
+F 5 "RMCF0805JT120RCT-ND" H 8000 2550 60  0001 C CNN "DigikeyPart"
 	1    8000 2550
 	-1   0    0    1
@@
 F 0 "JP1" H 6050 1750 60  0000 C CNN
 F 1 "JUMPER" H 6050 1620 40  0000 C CNN
+F 2 "SM1206" H 5990 1810 60  0001 C CNN
+F 4 "N/A" H 6050 1700 60  0001 C CNN "Part"
+F 5 "N/A" H 6050 1700 60  0001 C CNN "DigikeyPart"
 	1    6050 1700
 	1    0    0    -1
@@
 F 0 "D3" H 6250 3550 50  0000 C CNN
 F 1 "LED" H 6100 3400 50  0000 C CNN
+F 2 "LED-1206" H 6200 3600 60  0001 C CNN
+F 4 "APT3216SGC" H 6250 3450 60  0001 C CNN "Part"
+F 5 "754-1141-1-ND" H 6250 3450 60  0001 C CNN "DigikeyPart"
 	1    6250 3450
 	0    -1   -1   0
@@
 F 0 "D2" H 6000 3550 50  0000 C CNN
 F 1 "LED" H 5850 3400 50  0000 C CNN
+F 2 "LED-1206" H 5950 3600 60  0001 C CNN
+F 4 "APT3216SGC" H 6000 3450 60  0001 C CNN "Part"
+F 5 "754-1141-1-ND" H 6000 3450 60  0001 C CNN "DigikeyPart"
 	1    6000 3450
 	0    -1   -1   0
@@
 F 0 "R3" V 6330 3950 50  0000 C CNN
 F 1 "1K" V 6250 3950 50  0000 C CNN
+F 2 "SM0805" V 6380 3900 60  0001 C CNN
+F 4 "RMCF0805JT1K00" H 6250 3950 60  0001 C CNN "Part"
+F 5 "RMCF0805JT1K00CT-ND" H 6250 3950 60  0001 C CNN "DigikeyPart"
 	1    6250 3950
 	-1   0    0    1
@@
 F 0 "R2" V 6080 3950 50  0000 C CNN
 F 1 "1K" V 6000 3950 50  0000 C CNN
+F 2 "SM0805" V 6130 3900 60  0001 C CNN
+F 4 "RMCF0805JT1K00" H 6000 3950 60  0001 C CNN "Part"
+F 5 "RMCF0805JT1K00CT-ND" H 6000 3950 60  0001 C CNN "DigikeyPart"
 	1    6000 3950
 	-1   0    0    1
@@
 F 0 "C2" H 3550 2900 50  0000 L CNN
 F 1 "10uF" H 3450 2700 50  0000 L CNN
+F 2 "SM0805" H 3500 2950 60  0001 C CNN
+F 4 "TPSA106M010R1800" H 3550 2800 60  0001 C CNN "Part"
+F 5 "478-4086-1-ND" H 3550 2800 60  0001 C CNN "DigikeyPart"
 	1    3550 2800
 	1    0    0    -1
@@
 F 0 "C3" H 3850 3750 50  0000 L CNN
 F 1 "0.1uF" H 3850 3550 50  0000 L CNN
+F 2 "SM0805" H 3900 3800 60  0001 C CNN
+F 4 "CC0805ZRY5V9BB104" H 3800 3650 60  0001 C CNN "Part"
+F 5 "311-1361-1-ND" H 3800 3650 60  0001 C CNN "DigikeyPart"
 	1    3800 3650
 	1    0    0    -1
@@
 F 0 "C1" H 3200 2900 50  0000 L CNN
 F 1 "0.1uF" H 3200 2700 50  0000 L CNN
+F 2 "SM0805" H 3150 2950 60  0001 C CNN
+F 4 "CC0805ZRY5V9BB104" H 3300 2800 60  0001 C CNN "Part"
+F 5 "311-1361-1-ND" H 3300 2800 60  0001 C CNN "DigikeyPart"
 	1    3300 2800
 	1    0    0    -1
@@
 F 0 "J1" H 2775 2700 60  0000 C CNN
 F 1 "USB_2" H 2900 2150 60  0001 C CNN
-F 2 "VCC" H 3175 2600 50  0001 C CNN
-F 3 "D+" H 3150 2500 50  0001 C CNN
-F 4 "D-" H 3150 2400 50  0001 C CNN "Data-"
-F 5 "GND" H 3175 2300 50  0001 C CNN "Ground"
+F 2 "USB_MINI_A" H 2715 2760 50  0001 C CNN
+F 4 "896-43-005-00-100001" H 3150 2400 50  0001 C CNN "Part"
+F 5 "ED90342CT-ND" H 3175 2300 50  0001 C CNN "DigikeyPart"
 	1    2850 2450
 	1    0    0    -1
@@
 F 0 "U2" H 6840 3170 50  0000 L BNN
 F 1 "SN75176B" H 6840 2260 50  0000 L BNN
-F 2 "DIL8" H 7200 2750 50  0001 C CNN
+F 2 "SOIC8" H 7200 2750 50  0001 C CNN
+F 4 "SN75176BPSR" H 7550 2650 60  0001 C CNN "Part"
+F 5 "296-27995-1-ND" H 7550 2650 60  0001 C CNN "DigikeyPart"
 	1    7550 2650
 	1    0    0    -1
@@
 F 0 "U1" H 5300 2000 60  0000 C CNN
 F 1 "FT232RL" H 4900 3850 60  0000 C CNN
+F 2 "SSOP28" H 5360 1940 60  0001 C CNN
+F 4 "FT232RL-REEL" H 4900 2950 60  0001 C CNN "Part"
+F 5 "768-1007-1-ND" H 4900 2950 60  0001 C CNN "DigikeyPart"
 	1    4900 2950
 	1    0    0    -1

Commit message: finished ledmini, controller, and comm boards -- need to re-panelize myro boards
Parts:
- added FB1: FILTER, SM0603, symbol FILTER
Connections:
- net VCC: now also FB1.2; no longer J1.1
- new net: FB1.1, J1.1
Other:
- moved on the sheet: J1
Changed lines of the file:
@@
-EESchema Schematic File Version 2  date Mon 13 Jun 2011 01:48:36 AM EDT
+EESchema Schematic File Version 2  date Sun 07 Aug 2011 01:58:43 PM EDT
 LIBS:power
 LIBS:device
@@
 LIBS:SparkFun
 LIBS:commbrd-cache
-EELAYER 24  0
+EELAYER 25  0
 EELAYER END
 $Descr A4 11700 8267
+encoding utf-8
 Sheet 1 1
 Title ""
-Date "13 jun 2011"
+Date "7 aug 2011"
 Rev ""
 Comp ""
@@
 Comment4 ""
 $EndDescr
+Wire Wire Line
+	3050 2300 3550 2300
+Wire Wire Line
+	2300 2600 3050 2600
+Wire Wire Line
+	3050 2600 3050 3000
+Wire Wire Line
+	2850 3800 2850 3850
+Connection ~ 3450 2300
+Connection ~ 3450 3000
+Wire Wire Line
+	3950 2650 3850 2650
+Wire Wire Line
+	2300 2400 3950 2400
+Wire Wire Line
+	6350 1700 6550 1700
+Wire Wire Line
+	8600 3500 8250 3500
+Wire Wire Line
+	8250 3500 8250 2500
+Wire Wire Line
+	8250 2500 8600 2500
+Wire Wire Line
+	8600 3300 8350 3300
+Wire Wire Line
+	8350 3300 8350 2300
+Wire Wire Line
+	8350 2300 8600 2300
+Wire Wire Line
+	8600 3100 8450 3100
+Wire Wire Line
+	8450 3100 8450 2100
+Wire Wire Line
+	8450 2100 8600 2100
+Connection ~ 8550 1900
+Wire Wire Line
+	8600 2900 8550 2900
+Wire Wire Line
+	8550 2900 8550 1900
+Wire Wire Line
+	8600 1900 8000 1900
+Wire Wire Line
+	8000 1900 8000 2300
+Wire Wire Line
+	7750 2250 7750 2150
+Wire Wire Line
+	8000 2300 7900 2300
+Wire Wire Line
+	7900 2300 7900 2450
+Wire Wire Line
+	7900 2450 7750 2450
+Wire Wire Line
+	6550 1700 6550 2450
+Wire Wire Line
+	6550 2450 6650 2450
+Wire Wire Line
+	6650 2850 6500 2850
+Wire Wire Line
+	6500 2850 6500 2350
+Wire Wire Line
+	4900 4150 4900 4250
+Connection ~ 4900 4150
+Wire Wire Line
+	3800 3850 3800 3900
+Connection ~ 3300 3000
+Wire Wire Line
+	3050 3000 3550 3000
+Connection ~ 3100 3000
+Wire Wire Line
+	3100 3050 3100 3000
+Connection ~ 3100 2300
+Wire Wire Line
+	6450 4100 6450 4200
+Wire Wire Line
+	6450 4200 6000 4200
+Wire Wire Line
+	6000 3650 6000 3700
+Wire Wire Line
+	5800 3150 6250 3150
+Wire Wire Line
+	3850 2150 3850 2300
+Wire Wire Line
+	3850 2300 3950 2300
+Wire Wire Line
+	5800 3050 6000 3050
+Wire Wire Line
+	6000 3050 6000 3250
+Wire Wire Line
+	6250 3150 6250 3250
+Wire Wire Line
+	6250 3650 6250 3700
+Wire Wire Line
+	3100 2300 3100 2250
+Wire Wire Line
+	3950 2400 3950 2550
+Wire Wire Line
+	3300 2600 3300 2300
+Wire Wire Line
+	3550 2300 3550 2600
+Connection ~ 3300 2300
+Wire Wire Line
+	3950 3450 3800 3450
+Connection ~ 4750 4150
+Wire Wire Line
+	5200 4150 4600 4150
+Connection ~ 5050 4150
+Wire Wire Line
+	6650 2250 5800 2250
+Wire Wire Line
+	6650 2450 6650 2650
+Wire Wire Line
+	3950 2300 3950 2200
+Connection ~ 3950 2300
+Wire Wire Line
+	7750 2650 7900 2650
+Wire Wire Line
+	7900 2650 7900 2800
+Wire Wire Line
+	7750 2850 7750 2950
+Wire Wire Line
+	7900 2800 8100 2800
+Wire Wire Line
+	8100 2800 8100 2000
+Wire Wire Line
+	8100 2000 8600 2000
+Connection ~ 8000 2800
+Wire Wire Line
+	8500 2000 8500 3000
+Wire Wire Line
+	8500 3000 8600 3000
+Connection ~ 8500 2000
+Wire Wire Line
+	8600 2200 8400 2200
+Wire Wire Line
+	8400 2200 8400 3200
+Wire Wire Line
+	8400 3200 8600 3200
+Wire Wire Line
+	8600 2400 8300 2400
+Wire Wire Line
+	8300 2400 8300 3400
+Wire Wire Line
+	8300 3400 8600 3400
+Wire Wire Line
+	8600 3600 8200 3600
+Wire Wire Line
+	8200 3600 8200 2600
+Wire Wire Line
+	8200 2600 8600 2600
+Wire Wire Line
+	5750 1700 5700 1700
+Wire Wire Line
+	5700 1700 5700 1650
+Wire Wire Line
+	2300 2500 3850 2500
+Wire Wire Line
+	3850 2500 3850 2650
+Wire Wire Line
+	2850 2800 2850 2850
+Wire Wire Line
+	2850 3350 2850 3400
+Wire Wire Line
+	6500 2350 5800 2350
+Connection ~ 8000 2300
+Connection ~ 6650 2450
+Connection ~ 6500 2850
+Connection ~ 6600 2250
 Connection ~ 6250 4200
-Connection ~ 6600 2250
-Connection ~ 6500 2850
-Connection ~ 6650 2450
-Connection ~ 8000 2300
-Wire Wire Line
-	5800 2350 6500 2350
-Wire Wire Line
-	2850 3350 2850 3400
-Wire Wire Line
-	2850 2800 2850 2850
-Wire Wire Line
-	3850 2500 3850 2650
-Wire Wire Line
-	3850 2500 3050 2500
-Wire Wire Line
-	5700 1650 5700 1700
-Wire Wire Line
-	5700 1700 5750 1700
-Wire Wire Line
-	8600 2600 8200 2600
-Wire Wire Line
-	8200 2600 8200 3600
-Wire Wire Line
-	8200 3600 8600 3600
-Wire Wire Line
-	8600 3400 8300 3400
-Wire Wire Line
-	8300 3400 8300 2400
-Wire Wire Line
-	8300 2400 8600 2400
-Wire Wire Line
-	8600 3200 8400 3200
-Wire Wire Line
-	8400 3200 8400 2200
-Wire Wire Line
-	8400 2200 8600 2200
-Connection ~ 8500 2000
-Wire Wire Line
-	8600 3000 8500 3000
-Wire Wire Line
-	8500 3000 8500 2000
-Connection ~ 8000 2800
-Wire Wire Line
-	8600 2000 8100 2000
-Wire Wire Line
-	8100 2000 8100 2800
-Wire Wire Line
-	8100 2800 7900 2800
-Wire Wire Line
-	7750 2850 7750 2950
-Wire Wire Line
-	7900 2800 7900 2650
-Wire Wire Line
-	7900 2650 7750 2650
-Connection ~ 3950 2300
-Wire Wire Line
-	3950 2200 3950 2300
-Wire Wire Line
-	6650 2650 6650 2450
-Wire Wire Line
-	5800 2250 6650 2250
-Connection ~ 5050 4150
-Wire Wire Line
-	4600 4150 5200 4150
-Connection ~ 4750 4150
-Wire Wire Line
-	3950 3450 3800 3450
-Connection ~ 3300 2300
-Wire Wire Line
-	3550 2600 3550 2300
-Wire Wire Line
-	3550 2300 3050 2300
-Wire Wire Line
-	3300 2300 3300 2600
-Wire Wire Line
-	3950 2550 3950 2400
-Wire Wire Line
-	3100 2250 3100 2300
-Wire Wire Line
-	6250 3650 6250 3700
-Wire Wire Line
-	6250 3250 6250 3150
-Wire Wire Line
-	6000 3250 6000 3050
-Wire Wire Line
-	6000 3050 5800 3050
-Wire Wire Line
-	3950 2300 3850 2300
-Wire Wire Line
-	3850 2300 3850 2150
-Wire Wire Line
-	6250 3150 5800 3150
-Wire Wire Line
-	6000 3650 6000 3700
-Wire Wire Line
-	6000 4200 6450 4200
-Wire Wire Line
-	6450 4200 6450 4100
-Connection ~ 3100 2300
-Wire Wire Line
-	3100 3050 3100 3000
-Connection ~ 3100 3000
-Wire Wire Line
-	3050 2600 3050 3000
-Wire Wire Line
-	3050 3000 3550 3000
-Connection ~ 3300 3000
-Wire Wire Line
-	3800 3850 3800 3900
-Connection ~ 4900 4150
-Wire Wire Line
-	4900 4150 4900 4250
-Wire Wire Line
-	6500 2350 6500 2850
-Wire Wire Line
-	6500 2850 6650 2850
-Wire Wire Line
-	6650 2450 6550 2450
-Wire Wire Line
-	6550 2450 6550 1700
-Wire Wire Line
-	7750 2450 7900 2450
-Wire Wire Line
-	7900 2450 7900 2300
-Wire Wire Line
-	7900 2300 8000 2300
-Wire Wire Line
-	7750 2250 7750 2150
-Wire Wire Line
-	8000 2300 8000 1900
-Wire Wire Line
-	8000 1900 8600 1900
-Wire Wire Line
-	8550 1900 8550 2900
-Wire Wire Line
-	8550 2900 8600 2900
-Connection ~ 8550 1900
-Wire Wire Line
-	8600 2100 8450 2100
-Wire Wire Line
-	8450 2100 8450 3100
-Wire Wire Line
-	8450 3100 8600 3100
-Wire Wire Line
-	8600 2300 8350 2300
-Wire Wire Line
-	8350 2300 8350 3300
-Wire Wire Line
-	8350 3300 8600 3300
-Wire Wire Line
-	8600 2500 8250 2500
-Wire Wire Line
-	8250 2500 8250 3500
-Wire Wire Line
-	8250 3500 8600 3500
-Wire Wire Line
-	6550 1700 6350 1700
-Wire Wire Line
-	3950 2400 3050 2400
-Wire Wire Line
-	3850 2650 3950 2650
-Connection ~ 3450 3000
-Connection ~ 3450 2300
-Wire Wire Line
-	2850 3800 2850 3850
+Wire Wire Line
+	2300 2300 2350 2300
+$Comp
+L FILTER FB1
+U 1 1 4E3ED1CD
+P 2700 2300
+F 0 "FB1" H 2850 2450 60  0000 C CNN
+F 1 "FILTER" H 2600 2450 60  0000 C CNN
+F 2 "SM0603" H 2700 2300 60  0000 C CNN
+F 4 "MMZ1608D220C" H 2700 2300 60  0001 C CNN "Part"
+F 5 "445-6406-1-ND" H 2700 2300 60  0001 C CNN "DigikeyPart"
+	1    2700 2300
+	1    0    0    -1
+$EndComp
 $Comp
 L CONN_1 PTXD1
@@
 L USB_2 J1
 U 1 1 4DE311C4
-P 2850 2450
-F 0 "J1" H 2775 2700 60  0000 C CNN
-F 1 "USB_2" H 2900 2150 60  0001 C CNN
-F 2 "USB_MINI_A" H 2715 2760 50  0001 C CNN
-F 4 "896-43-005-00-100001" H 3150 2400 50  0001 C CNN "Part"
-F 5 "ED90342CT-ND" H 3175 2300 50  0001 C CNN "DigikeyPart"
-	1    2850 2450
-	1    0    0    -1
-$EndComp
+P 2100 2450
+F 0 "J1" H 2025 2700 60  0000 C CNN
+F 1 "USB_2" H 2150 2150 60  0001 C CNN
+F 2 "USB_MINI_A" H 1965 2760 50  0001 C CNN
+F 4 "896-43-005-00-100001" H 2400 2400 50  0001 C CNN "Part"
+F 5 "ED90342CT-ND" H 2425 2300 50  0001 C CNN "DigikeyPart"
+	1    2100 2450
+	1    0    0    -1
+$EndComp
